File: Motor Cape/level_shifters.sch (KiCad schematic (older format))
At the start: 36 parts

Commit message: fixed drc errors, added serial comm between pi & due, now just need to choose power connector & fuse
Parts:
- gave numbers to parts that had none: 24
- renumbered back_left_A to back_left_A1, back_left_B to back_left_B1, back_right_A to back_right_A1, back_right_B to back_right_B1, draw_bridge_A to draw_bridge_A1, draw_bridge_B to draw_bridge_B1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
