File: Electrical/Motor Cape/level_shifters.sch (KiCad schematic (older format))
At the start: 36 parts

Commit message: worked more on motor cape
Parts:
- removed R1, R10, R11, R12, R13, R14, R15, R16, R17, R18, R19, R2, R20, R21, R22, R23, R24, R3, R4, R5, R6, R7, R8, R9: 10k, symbol R
- removed back_left_A1, back_left_B1, back_right_A1, back_right_B1, draw_bridge_A1, draw_bridge_B1, flag_wheel_A1, flag_wheel_B1, front_left_A1, front_left_B1, front_right_A1, front_right_B1: NFET, symbol Q_NMOS_DGS
