File: Electrical/Motor Cape/MotorCape.sch (KiCad schematic (older format))
At the start: 25 parts, among them J1 back_right motor, J11 flag_wheel servo, J2 front_right motor, J3 back_left motor, J4 front_left motor, J5 draw_bridge motor, J6 flag_wheel motor, J7 i2c bus connector, P1 Shifter_Front_HI, P10 Controller 2_2, P11 Controller 3_1, P12 Controller 3_2, P13 battery stuff, P14 CONN_01X04, P2 Shifter_Front_LO, P3 Shifter_Back_HI, P4 Shifter_Back_LO, P5 Shifter_Misc_HI, P6 Shifter_Misc_LO, P7 Controller 1_1, P8 Controller 1_2, P9 Controller 2_1, U1 IMU

Commit message: added newest rules 3.3-1 stuff
Parts:
- removed ARD1: Arduino_Due_Shield, MotorCapeComponents:Arduino_Due_Shield, symbol Arduino_Due_Shield
- added ARD1: Arduino_Due_Shield-NEW, MotorCapeComponents:Arduino_Due_Shield, symbol Arduino_Due_Shield-NEW
- J1, J2, J3, J4, J5, J6: footprint Pin_Headers:Pin_Header_Angled_1x06_Pitch2.54mm -> Pin_Headers:Pin_Header_Straight_1x06
- J11: footprint Pin_Headers:Pin_Header_Angled_1x03_Pitch2.54mm -> Pin_Headers:Pin_Header_Straight_1x03
Connections:
- net +5V: now also ARD1.5 (5V)
- net Earth: now also ARD1.6 (GND)
- net FROM_Pi: now also ARD1.42 (D0_RX0)
- net SCL: now also ARD1.25 (SCL1)
- net SDA: now also ARD1.26 (SDA1)
- net TO_Pi: now also ARD1.41 (D1_TX0)
- net at J11.3 (Pin_3): now also ARD1.34 (D8)
- net at P2.1 (P1): now also ARD1.55 (D24)
- net at P2.2 (P2): now also ARD1.54 (D23)
- net at P2.5 (P5): now also ARD1.61 (D30)
- net at P2.6 (P6): now also ARD1.60 (D29)
- net at P4.1 (P1): now also ARD1.58 (D27)
- net at P4.2 (P2): now also ARD1.57 (D26)
- net at P4.5 (P5): now also ARD1.64 (D33)
- net at P4.6 (P6): now also ARD1.63 (D32)
- net at P6.1 (P1): now also ARD1.70 (D39)
- net at P6.2 (P2): now also ARD1.69 (D38)
- net at P6.5 (P5): now also ARD1.67 (D36)
- net at P6.6 (P6): now also ARD1.66 (D35)
- net at P7.1 (P1): now also ARD1.59 (D28)
- net at P7.2 (P2): now also ARD1.38 (D4_CS1)
- net at P7.3 (P3): now also ARD1.62 (D31)
- net at P7.4 (P4): now also ARD1.37 (D5)
- net at P9.2 (P2): now also ARD1.39 (D3)
- net at P9.3 (P3): now also ARD1.56 (D25)
- net at P9.4 (P4): now also ARD1.40 (D2)
- net at P9.5 (P5): now also ARD1.53 (D22)
- net at P11.2 (P2): now also ARD1.35 (D7)
- net at P11.3 (P3): now also ARD1.68 (D37)
- net at P11.4 (P4): now also ARD1.36 (D6)
- net at P11.5 (P5): now also ARD1.65 (D34)
Changed lines of the file:
@@
 LIBS:MotorCapeComponents
 LIBS:arduino
+LIBS:DueShieldComponents
 LIBS:MotorCape-cache
 EELAYER 25 0
@@
 $Descr A4 11693 8268
 encoding utf-8
-Sheet 1 2
+Sheet 1 1
 Title ""
 Date ""
@@
 F 0 "J1" H 9750 6300 50  0000 C CNN
 F 1 "back_right motor" H 9750 5600 50  0000 C CNN
-F 2 "Pin_Headers:Pin_Header_Angled_1x06_Pitch2.54mm" H 9750 6000 50  0001 C CNN
+F 2 "Pin_Headers:Pin_Header_Straight_1x06" H 9750 6000 50  0001 C CNN
 F 3 "" H 9750 6000 50  0001 C CNN
 	1    9750 6000
@@
 F 0 "J2" H 10950 5450 50  0000 C CNN
 F 1 "front_right motor" H 10950 4750 50  0000 C CNN
-F 2 "Pin_Headers:Pin_Header_Angled_1x06_Pitch2.54mm" H 10950 5150 50  0001 C CNN
+F 2 "Pin_Headers:Pin_Header_Straight_1x06" H 10950 5150 50  0001 C CNN
 F 3 "" H 10950 5150 50  0001 C CNN
 	1    10950 5150
@@
 F 0 "J3" H 2950 5350 50  0000 C CNN
 F 1 "back_left motor" H 2950 4650 50  0000 C CNN
-F 2 "Pin_Headers:Pin_Header_Angled_1x06_Pitch2.54mm" H 2950 5050 50  0001 C CNN
+F 2 "Pin_Headers:Pin_Header_Straight_1x06" H 2950 5050 50  0001 C CNN
 F 3 "" H 2950 5050 50  0001 C CNN
 	1    2950 5050
@@
 F 0 "J4" H 2950 4500 50  0000 C CNN
 F 1 "front_left motor" H 2950 3800 50  0000 C CNN
-F 2 "Pin_Headers:Pin_Header_Angled_1x06_Pitch2.54mm" H 2950 4200 50  0001 C CNN
+F 2 "Pin_Headers:Pin_Header_Straight_1x06" H 2950 4200 50  0001 C CNN
 F 3 "" H 2950 4200 50  0001 C CNN
 	1    2950 4200
@@
 F 0 "J6" H 2950 7300 50  0000 C CNN
 F 1 "flag_wheel motor" H 2900 6600 50  0000 C CNN
-F 2 "Pin_Headers:Pin_Header_Angled_1x06_Pitch2.54mm" H 2950 7000 50  0001 C CNN
+F 2 "Pin_Headers:Pin_Header_Straight_1x06" H 2950 7000 50  0001 C CNN
 F 3 "" H 2950 7000 50  0001 C CNN
 	1    2950 7000
@@
 F 0 "J5" H 2950 6400 50  0000 C CNN
 F 1 "draw_bridge motor" H 2950 5700 50  0000 C CNN
-F 2 "Pin_Headers:Pin_Header_Angled_1x06_Pitch2.54mm" H 2950 6100 50  0001 C CNN
+F 2 "Pin_Headers:Pin_Header_Straight_1x06" H 2950 6100 50  0001 C CNN
 F 3 "" H 2950 6100 50  0001 C CNN
 	1    2950 6100
@@
 F 0 "J11" H 8700 3950 50  0000 C CNN
 F 1 "flag_wheel servo" H 8700 3550 50  0000 C CNN
-F 2 "Pin_Headers:Pin_Header_Angled_1x03_Pitch2.54mm" H 8700 3750 50  0001 C CNN
+F 2 "Pin_Headers:Pin_Header_Straight_1x03" H 8700 3750 50  0001 C CNN
 F 3 "" H 8700 3750 50  0001 C CNN
 	1    8700 3750
@@
 	9300 4200 9300 4350
 $Comp
-L Arduino_Due_Shield ARD1
-U 1 1 5A993409
-P 5850 2400
-F 0 "ARD1" V 5950 2400 60  0000 C CNN
-F 1 "Arduino_Due_Shield" V 5750 2400 60  0000 C CNN
-F 2 "MotorCapeComponents:Arduino_Due_Shield" H 6550 5150 60  0001 C CNN
-F 3 "" H 6550 5150 60  0001 C CNN
-	1    5850 2400
-	0    1    1    0
-$EndComp
-$Comp
 L CONN_01X04 P14
 U 1 1 5AA1DD33
@@
 NoConn ~ 8450 2350
 NoConn ~ 8450 2650
-$Comp
-L IMU U1
-U 1 1 5AA1F45A
-P 9250 2200
-F 0 "U1" H 9650 2250 60  0000 C CNN
-F 1 "IMU" H 9650 2350 60  0000 C CNN
-F 2 "MotorCapeComponents:IMU" H 9250 2200 60  0001 C CNN
-F 3 "" H 9250 2200 60  0000 C CNN
-	1    9250 2200
-	1    0    0    -1
-$EndComp
 $Comp
 L Earth #PWR042
@@
 SCL
 $Comp
-L +3.3V #PWR?
+L +3.3V #PWR044
 U 1 1 5AAB580D
 P 8950 3000
-F 0 "#PWR?" H 8950 2850 50  0001 C CNN
+F 0 "#PWR044" H 8950 2850 50  0001 C CNN
 F 1 "+3.3V" H 8950 3140 50  0000 C CNN
 F 2 "" H 8950 3000 50  0000 C CNN
@@
 $EndComp
 $Comp
-L +3.3V #PWR?
+L +3.3V #PWR045
 U 1 1 5AAB58EE
 P 8950 2750
-F 0 "#PWR?" H 8950 2600 50  0001 C CNN
+F 0 "#PWR045" H 8950 2600 50  0001 C CNN
 F 1 "+3.3V" H 8950 2890 50  0000 C CNN
 F 2 "" H 8950 2750 50  0000 C CNN
@@
 Wire Wire Line
 	9050 2750 8950 2750
+$Comp
+L IMU U1
+U 1 1 5ABDC0C0
+P 9250 2200
+F 0 "U1" H 9650 2250 60  0000 C CNN
+F 1 "IMU" H 9650 2350 60  0000 C CNN
+F 2 "MotorCapeComponents:IMU" H 9250 2200 60  0001 C CNN
+F 3 "" H 9250 2200 60  0000 C CNN
+	1    9250 2200
+	1    0    0    -1
+$EndComp
+$Comp
+L Arduino_Due_Shield-NEW ARD1
+U 1 1 5ABDC643
+P 5850 2400
+F 0 "ARD1" V 5950 2400 60  0000 C CNN
+F 1 "Arduino_Due_Shield-NEW" V 5750 2400 60  0000 C CNN
+F 2 "MotorCapeComponents:Arduino_Due_Shield" H 6550 5150 60  0001 C CNN
+F 3 "" H 6550 5150 60  0001 C CNN
+	1    5850 2400
+	0    1    1    0
+$EndComp
 $EndSCHEMATC
