File: Electrical/Motor Cape/MotorCape.kicad_pcb (KiCad board)
At the start: 2 copper layers, 15 parts, among them J9 Raspberry_Pi_2_3, P1 Shifter_Front_HI, P10 Controller 2_2, P11 Controller 3_1, P12 Controller 3_2, P13 battery stuff, P2 Shifter_Front_LO, P3 Shifter_Back_HI, P4 Shifter_Back_LO, P5 Shifter_Misc_HI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

Commit message: added newest rules 3.3-1 stuff
Parts:
- removed J9: Raspberry_Pi_2_3, Pin_Headers:Pin_Header_Straight_2x20
- added F1: Fuse, Fuse_Holders_and_Fuses:Fuseholder5x20_horiz_open_inline_Type-I, F.Cu at (67.0, 103.5)
- added J1: back_right motor, Pin_Headers:Pin_Header_Straight_1x06, F.Cu at (97.0, 67.5)
- added J11: flag_wheel servo, Pin_Headers:Pin_Header_Straight_1x03, F.Cu at (21.0, 87.5)
- added J2: front_right motor, Pin_Headers:Pin_Header_Straight_1x06, F.Cu at (134.5, 115.0)
- added J3: back_left motor, Pin_Headers:Pin_Header_Straight_1x06, F.Cu at (119.5, 115.0)
- added J4: front_left motor, Pin_Headers:Pin_Header_Straight_1x06, F.Cu at (124.5, 111.0)
- added J5: draw_bridge motor, Pin_Headers:Pin_Header_Straight_1x06, F.Cu at (21.0, 87.5)
- added J6: flag_wheel motor, Pin_Headers:Pin_Header_Straight_1x06, F.Cu at (21.0, 87.5)
- added J7: i2c bus connector, Pin_Headers:Pin_Header_Straight_1x02, F.Cu at (69.0, 71.5)
- added P14: CONN_01X04, Pin_Headers:Pin_Header_Straight_1x04, F.Cu at (117.5, 82.5)
- added U1: IMU, MotorCapeComponents:IMU, F.Cu at (97.0, 81.0)
- ARD1: value Arduino_Due_Shield -> Arduino_Due_Shield-NEW
- moved P12 187.1 mm to (48.2, 127.2), turned to 90 degrees
- moved P11 179.6 mm to (56.8, 127.2), turned to 180 degrees
- moved P10 170.3 mm to (48.5, 108.5), turned to 90 degrees
- moved P9 163.8 mm to (57.0, 108.5), turned to 180 degrees
- moved P8 153.5 mm to (48.5, 90.0), turned to 90 degrees
- moved P7 147.0 mm to (57.0, 90.0), turned to 180 degrees
- moved P2 97.7 mm to (147.5, 97.1), turned to 270 degrees
- moved P1 82.7 mm to (134.7, 107.0), turned to 90 degrees
- moved P13 80.2 mm to (64.5, 106.0)
- moved P4 72.5 mm to (119.5, 97.1), turned to 270 degrees
- moved P6 62.2 mm to (91.8, 107.8), turned to 270 degrees
- moved P3 55.9 mm to (106.7, 107.0), turned to 90 degrees
- moved P5 47.0 mm to (78.9, 117.7), turned to 90 degrees
- moved ARD1 37.0 mm to (61.6, 75.6)
Connections:
- ARD1 pad 1: Net-(ARD1-Pad1) -> (no net)
- ARD1 pad 10: Net-(ARD1-Pad10) -> (no net)
- ARD1 pad 11: Net-(ARD1-Pad11) -> (no net)
- ARD1 pad 12: Net-(ARD1-Pad12) -> (no net)
- ARD1 pad 13: Net-(ARD1-Pad13) -> (no net)
- ARD1 pad 14: Net-(ARD1-Pad14) -> (no net)
- ARD1 pad 15: Net-(ARD1-Pad15) -> (no net)
- ARD1 pad 16: Net-(ARD1-Pad16) -> (no net)
- ARD1 pad 17: Net-(ARD1-Pad17) -> (no net)
- ARD1 pad 18: Net-(ARD1-Pad18) -> (no net)
- ARD1 pad 19: Net-(ARD1-Pad19) -> (no net)
- ARD1 pad 2: Net-(ARD1-Pad2) -> (no net)
- ARD1 pad 20: Net-(ARD1-Pad20) -> (no net)
- ARD1 pad 21: Net-(ARD1-Pad21) -> (no net)
- ARD1 pad 22: Net-(ARD1-Pad22) -> (no net)
- ARD1 pad 23: Net-(ARD1-Pad23) -> (no net)
- ARD1 pad 24: Net-(ARD1-Pad24) -> (no net)
- ARD1 pad 27: Net-(ARD1-Pad27) -> (no net)
- ARD1 pad 28: Net-(ARD1-Pad28) -> (no net)
- ARD1 pad 29: Net-(ARD1-Pad29) -> (no net)
- ARD1 pad 3: Net-(ARD1-Pad3) -> (no net)
- ARD1 pad 30: Net-(ARD1-Pad30) -> (no net)
- ARD1 pad 31: Net-(ARD1-Pad31) -> (no net)
- ARD1 pad 32: Net-(ARD1-Pad32) -> (no net)
- ARD1 pad 33: Net-(ARD1-Pad33) -> (no net)
- ARD1 pad 4: Net-(ARD1-Pad4) -> (no net)
- ARD1 pad 43: Net-(ARD1-Pad43) -> (no net)
- ARD1 pad 44: Net-(ARD1-Pad44) -> (no net)
- ARD1 pad 45: Net-(ARD1-Pad45) -> (no net)
- ARD1 pad 46: Net-(ARD1-Pad46) -> (no net)
- ARD1 pad 47: Net-(ARD1-Pad47) -> (no net)
- ARD1 pad 48: Net-(ARD1-Pad48) -> (no net)
- ARD1 pad 49: Net-(ARD1-Pad49) -> (no net)
- ARD1 pad 5: Net-(ARD1-Pad5) -> +5V
- ARD1 pad 50: Net-(ARD1-Pad50) -> (no net)
- ARD1 pad 51: Net-(ARD1-Pad51) -> (no net)
- ARD1 pad 52: Net-(ARD1-Pad52) -> (no net)
- ARD1 pad 6: Net-(ARD1-Pad6) -> Earth
- ARD1 pad 7: Net-(ARD1-Pad7) -> (no net)
- ARD1 pad 71: Net-(ARD1-Pad71) -> (no net)
- ARD1 pad 72: Net-(ARD1-Pad72) -> (no net)
- ARD1 pad 73: Net-(ARD1-Pad73) -> (no net)
- ARD1 pad 74: Net-(ARD1-Pad74) -> (no net)
- ARD1 pad 75: Net-(ARD1-Pad75) -> (no net)
- ARD1 pad 76: Net-(ARD1-Pad76) -> (no net)
- ARD1 pad 77: Net-(ARD1-Pad77) -> (no net)
- ARD1 pad 78: Net-(ARD1-Pad78) -> (no net)
- ARD1 pad 79: Net-(ARD1-Pad79) -> (no net)
- ARD1 pad 8: Net-(ARD1-Pad8) -> (no net)
- ARD1 pad 80: Net-(ARD1-Pad80) -> (no net)
- ARD1 pad 81: Net-(ARD1-Pad81) -> (no net)
- ARD1 pad 82: Net-(ARD1-Pad82) -> (no net)
- ARD1 pad 83: Net-(ARD1-Pad83) -> (no net)
- ARD1 pad 84: Net-(ARD1-Pad84) -> (no net)
- ARD1 pad 85: Net-(ARD1-Pad85) -> (no net)
- ARD1 pad 86: Net-(ARD1-Pad86) -> (no net)
- ARD1 pad 87: Net-(ARD1-Pad87) -> (no net)
- ARD1 pad 88: Net-(ARD1-Pad88) -> (no net)
- ARD1 pad 89: Net-(ARD1-Pad89) -> (no net)
- ARD1 pad 9: Net-(ARD1-Pad9) -> (no net)
- ARD1 pad 90: Earth -> (no net)
- ARD1 pad 91: Net-(ARD1-Pad91) -> (no net)
- ARD1 pad 92: +5V -> (no net)

Commit message: initialized shell for relative heading for indoors
Parts:
- moved J11 13.3 mm to (27.4, 75.8)
- moved J6 8.76 mm to (29.8, 88.0)
- moved J5 4.00 mm to (18.6, 90.7)
Changed lines of the file:
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@@
   (general
     (links 98)
-    (no_connects 96)
-    (area 0 0 0 0)
+    (no_connects 98)
+    (area 13.724999 60.820237 163.494001 133.325)
     (thickness 1.6)
     (drawings 24)
@@
   )
   (module Pin_Headers:Pin_Header_Straight_1x06 (layer F.Cu)
-    (at 21 87.5)
+    (at 18.6 90.7)
     (descr "Through hole pin header")
     (tags "pin header")
@@
   )
   (module Pin_Headers:Pin_Header_Straight_1x06 (layer F.Cu)
-    (at 21 87.5)
+    (at 29.75 88)
     (descr "Through hole pin header")
     (tags "pin header")
@@
   )
   (module Pin_Headers:Pin_Header_Straight_1x03 (layer F.Cu)
-    (at 21 87.5)
-    (descr "Through hole pin header")
-    (tags "pin header")
+    (at 27.35 75.85)
+    (descr "Through hole pin header")
+    (tags "pin header")
