File: Electrical/Pi Cape/i2c0.sch (KiCad schematic (older format))
At the start: 1 part, among them J1 Dist_Sensor

Commit message: finished footprints on Pi cape. onto layouts
Parts:
- J1: footprint (none) -> Pi Cape Footprints:Pin_Header_Latched_1x05
Changed lines of the file:
@@
 AR Path="/5AAB9EF4/5AAB6BB2/5AAB57E4" Ref="J7"  Part="1"
 AR Path="/5AAB9EF4/5AAB6BB7/5AAB57E4" Ref="J8"  Part="1"
-F 0 "J1" H 2850 1650 50  0000 C CNN
+F 0 "J6" H 2850 1650 50  0000 C CNN
 F 1 "Dist_Sensor" V 2950 1350 50  0000 C CNN
-F 2 "" H 2850 1350 50  0001 C CNN
+F 2 "Pi Cape Footprints:Pin_Header_Latched_1x05" H 2850 1350 50  0001 C CNN
 F 3 "" H 2850 1350 50  0001 C CNN
 	1    2850 1350

Commit message: updated pi cape to have 7-seg and spaced components in layout
Changed lines of the file:
@@
 AR Path="/5AAB9EF4/5AAB6BB2/5AAB57E4" Ref="J7"  Part="1"
 AR Path="/5AAB9EF4/5AAB6BB7/5AAB57E4" Ref="J8"  Part="1"
-F 0 "J6" H 2850 1650 50  0000 C CNN
+F 0 "J1" H 2850 1650 50  0000 C CNN
 F 1 "Dist_Sensor" V 2950 1350 50  0000 C CNN
 F 2 "Pi Cape Footprints:Pin_Header_Latched_1x05" H 2850 1350 50  0001 C CNN

Commit message: added newest rules 3.3-1 stuff
Changed lines of the file:
@@
 AR Path="/5AAB9EF4/5AAB6BB2/5AAB57E4" Ref="J7"  Part="1"
 AR Path="/5AAB9EF4/5AAB6BB7/5AAB57E4" Ref="J8"  Part="1"
-F 0 "J1" H 2850 1650 50  0000 C CNN
+F 0 "J7" H 2850 1650 50  0000 C CNN
 F 1 "Dist_Sensor" V 2950 1350 50  0000 C CNN
 F 2 "Pi Cape Footprints:Pin_Header_Latched_1x05" H 2850 1350 50  0001 C CNN
