File: Electrical/MotorCape_hierchal/MotorCape.kicad_pcb (KiCad board)
At the start: 2 copper layers, 152.4 x 56.4 mm, 23 parts, among them P13 battery_connector, U1 IMU

Commit message: successfully tested all encoders on motor controller board
Other:
- board text added: "22"
- board text added: "26"
- board text added: "30"
- board text added: "34"
- board text added: "38"
- board text added: "42"
- board text added: "46"
- board text added: "50"
- board text added: "5V"
- board text added: "GND"
Changed lines of the file:
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@@
-(kicad_pcb (version 4) (host pcbnew 4.0.6)
+(kicad_pcb (version 4) (host pcbnew 4.0.5)
   (general
     (links 110)
@@
     (area 50.6836 65.456999 203.541701 121.995001)
     (thickness 1.6)
-    (drawings 5)
+    (drawings 15)
     (tracks 1229)
     (zones 0)
@@
     )
   )
+  (gr_text 5V (at 193.04 69.215) (layer F.Fab)
+    (effects (font (size 1.5 1.5) (thickness 0.3)))
+  )
+  (gr_text GND (at 191.77 112.395) (layer F.Fab)
+    (effects (font (size 1.5 1.5) (thickness 0.3)))
+  )
+  (gr_text 50 (at 193.04 107.315) (layer F.Fab)
+    (effects (font (size 1.5 1.5) (thickness 0.3)))
+  )
+  (gr_text 46 (at 193.04 102.235) (layer F.Fab)
+    (effects (font (size 1.5 1.5) (thickness 0.3)))
+  )
+  (gr_text 42 (at 193.04 97.155) (layer F.Fab)
+    (effects (font (size 1.5 1.5) (thickness 0.3)))
+  )
+  (gr_text 38 (at 193.04 92.075) (layer F.Fab)
+    (effects (font (size 1.5 1.5) (thickness 0.3)))
+  )
+  (gr_text 34 (at 193.04 86.995) (layer F.Fab)
+    (effects (font (size 1.5 1.5) (thickness 0.3)))
+  )
+  (gr_text 30 (at 193.04 81.915) (layer F.Fab)
+    (effects (font (size 1.5 1.5) (thickness 0.3)))
+  )
+  (gr_text 26 (at 193.04 76.835) (layer F.Fab)
+    (effects (font (size 1.5 1.5) (thickness 0.3)))
+  )
+  (gr_text 22 (at 193.04 71.755) (layer F.Fab)
+    (effects (font (size 1.5 1.5) (thickness 0.3)))
+  )
   (gr_text "GT IEEE Hardware Team 2017-2018" (at 73.406 116.586) (layer F.SilkS)
